Commit message: [mc_env_description] add OmniWalls.urdf

File: mc_env_description/urdf/SideWalls.urdf (robot description, URDF)
Before this commit: robot SideWalls, 3 links, 2 joints
Joints:
- joint LeftWall: origin xyz=0.0 0.0 0.0 rpy=0.0 -0.0 0.0 -> xyz=0.0 1.0 1.0 rpy=0.0 0.0 0.0
- joint RightWall: origin xyz=0.0 0.0 0.0 rpy=0.0 -0.0 0.0 -> xyz=0.0 -1.0 1.0 rpy=0.0 0.0 0.0
