Commit message: [mc_env_description] update urdf/TiltedScaffold.urdf

File: mc_env_description/urdf/TiltedScaffold.urdf (robot description, URDF)
Before this commit: robot TiltedScaffold, 3 links, 2 joints
Links:
- link RightGroundBlock: geometry collision box size=0.25 0.25 0.02; visual box size=0.25 0.25 0.02
Joints:
- joint LeftWall: origin xyz=0.3 0.7 1.0 rpy=0 0 0 -> xyz=0.35 0.7 1.5 rpy=0 0 0
- joint RightGroundBlock: origin xyz=0.3 -0.2 0.1 rpy=-0.349 0 0 -> xyz=0.35 -0.2 0.1 rpy=-0.349 0 0

Commit message: [mc_env_description] update urdf/TiltedScaffold.urdf

File: mc_env_description/urdf/TiltedScaffold.urdf (robot description, URDF)
Before this commit: robot TiltedScaffold, 3 links, 2 joints
Links:
- added link LeftGroundBlock; collision box size=0.25 0.25 0.02; visual box size=0.25 0.25 0.02
- added link RightWall; collision box size=0.2 0.02 0.2; visual box size=0.2 0.02 0.2
Joints:
- added joint LeftGroundBlock: type fixed, parent base_link, child LeftGroundBlock, origin xyz=1.25 0.2 0.1 rpy=0.5236 0 0
- added joint RightWall: type fixed, parent base_link, child RightWall, origin xyz=1.25 -0.7 1.5 rpy=0 0 0
- joint RightGroundBlock: origin xyz=0.35 -0.2 0.1 rpy=-0.349 0 0 -> xyz=0.35 -0.2 0.1 rpy=-0.5236 0 0

Commit message: [mc_env_description] update urdf/TiltedScaffold.urdf

File: mc_env_description/urdf/TiltedScaffold.urdf (robot description, URDF)
Before this commit: robot TiltedScaffold, 5 links, 4 joints
Joints:
- joint LeftGroundBlock: origin xyz=1.25 0.2 0.1 rpy=0.5236 0 0 -> xyz=1.25 0.2 0.1 rpy=0.4363 0 0
- joint RightGroundBlock: origin xyz=0.35 -0.2 0.1 rpy=-0.5236 0 0 -> xyz=0.35 -0.2 0.1 rpy=-0.4363 0 0
