Commit message: Add an position offset to the fixed joint for mesh shape.

File: mc_env_description/urdf/ground.urdf (robot description, URDF)
Before this commit: robot ground, 2 links, 1 joints
Joints:
- joint ground: origin xyz=0.0 0.0 0.0 rpy=0.0 -0.0 0.0 -> xyz=20.0 0.0 0.0 rpy=0.0 0.0 0.0

Commit message: Add an position offset to the fixed joint for box shape.

File: mc_env_description/urdf/ground.urdf (robot description, URDF)
Before this commit: robot ground, 2 links, 1 joints
Links:
- link ground: geometry collision box size=20.0 20.0 0.1; visual box size=20.0 20.0 0.1
Joints:
- joint ground: origin xyz=0.0 0.0 0.0 rpy=0.0 -0.0 0.0 -> xyz=20.0 0.0 0.0 rpy=0.0 0.0 0.0

Commit message: Add an position offset to the geometry for box shape.

File: mc_env_description/urdf/ground.urdf (robot description, URDF)
Before this commit: robot ground, 2 links, 1 joints
Links:
- link ground: geometry collision box size=20.0 20.0 0.1; visual box size=20.0 20.0 0.1
