Commit message: Add the dummy joints and links for tactile sensors.

File: jvrc_description/urdf/jvrc1.urdf (robot description, URDF)
Before this commit: robot jvrc1, 60 links, 59 joints
Links:
- added link jvrc1_back_tactile_sensor
- added link jvrc1_left_foot_tactile_sensor
- added link jvrc1_left_knee_tactile_sensor
- added link jvrc1_left_thigh_tactile_sensor
- added link jvrc1_right_elbow_tactile_sensor
- added link jvrc1_right_foot_tactile_sensor
- added link jvrc1_right_thigh_tactile_sensor
Joints:
- added joint jvrc1_back_tactile_sensor: type fixed, parent WAIST_R_S, child jvrc1_back_tactile_sensor, origin xyz=-0.075 0.0 0.2 rpy=0.0 1.44 0.0
- added joint jvrc1_left_foot_tactile_sensor: type fixed, parent L_ANKLE_P_S, child jvrc1_left_foot_tactile_sensor, origin xyz=0.030310330912470818 -0.001216750591993332 -0.10773589462041855 rpy=0 0 0
- added joint jvrc1_left_knee_tactile_sensor: type fixed, parent L_KNEE_S, child jvrc1_left_knee_tactile_sensor, origin xyz=0.11161884184098951 -3.042248147844262e-09 -0.1063933713699532 rpy=3.141590255540823 -1.5204375874732723 -3.1415901265290733
- added joint jvrc1_left_thigh_tactile_sensor: type fixed, parent L_HIP_Y_S, child jvrc1_left_thigh_tactile_sensor, origin xyz=-0.0677307381928566 0 -0.20450757563611333 rpy=0 1.5242809442976415 0
- added joint jvrc1_right_elbow_tactile_sensor: type fixed, parent R_ELBOW_P_S, child jvrc1_right_elbow_tactile_sensor, origin xyz=-0.06975397769348207 0 -0.0720193897773116 rpy=0 1.5708 0
- added joint jvrc1_right_foot_tactile_sensor: type fixed, parent R_ANKLE_P_S, child jvrc1_right_foot_tactile_sensor, origin xyz=0.030310330912470818 -0.001216750591993332 -0.10773589462041855 rpy=0 0 0
- added joint jvrc1_right_thigh_tactile_sensor: type fixed, parent R_HIP_Y_S, child jvrc1_right_thigh_tactile_sensor, origin xyz=-0.0677307381928566 0 -0.20450757563611333 rpy=0 1.5242809442976415 0

Commit message: Update thigh tactile sensor frame.

File: jvrc_description/urdf/jvrc1.urdf (robot description, URDF)
Before this commit: robot jvrc1, 67 links, 66 joints
Joints:
- joint jvrc1_left_thigh_tactile_sensor: origin xyz=-0.0677307381928566 0 -0.20450757563611333 rpy=0 1.5242809442976415 0 -> xyz=-0.0677307381928566 0 -0.17450757563611333 rpy=0 1.5242809442976415 0
- joint jvrc1_right_thigh_tactile_sensor: origin xyz=-0.0677307381928566 0 -0.20450757563611333 rpy=0 1.5242809442976415 0 -> xyz=-0.0677307381928566 0 -0.17450757563611333 rpy=0 1.5242809442976415 0
